Commit message: yes
dw

File: src/fmauch_universal_robot/ur_description/urdf/inc/ur3e_macro.xacro (robot description, xacro)
@@ -17,5 +17,9 @@
           real robot.
   -->
+<<<<<<< HEAD
   <!-- <xacro:arg name="z_h" default="$(arg z_height)" /> -->
+=======
+  <xacro:arg name="z_h" default="$(arg z_height)" />
+>>>>>>> 9e3fc93 (yes)
   <xacro:macro name="ur3e_robot" params="
    prefix
@@ -30,5 +34,9 @@
   >
     <xacro:include filename="$(find ur_description)/urdf/inc/ur_macro.xacro">
+<<<<<<< HEAD
       <!-- <xacro:arg name="z_h" default="$(arg z_h)" /> -->
+=======
+      <xacro:arg name="z_h" default="$(arg z_h)" />
+>>>>>>> 9e3fc93 (yes)
     </xacro:include>
     <xacro:ur_robot

File: src/fmauch_universal_robot/ur_description/urdf/inc/ur_macro.xacro (robot description, xacro)
@@ -44,4 +44,5 @@
   <xacro:include filename="$(find ur_description)/urdf/inc/ur_transmissions.xacro" />
   <xacro:include filename="$(find ur_description)/urdf/inc/ur_common.xacro" />
+<<<<<<< HEAD
   <!-- robotiq_hande_gripper -->
   <xacro:include filename="$(find robotiq_description)/urdf/robotiq_hande_gripper.urdf.xacro" />
@@ -49,4 +50,8 @@
     prefix
     gripper
+=======
+  <xacro:macro name="ur_robot" params="
+    prefix
+>>>>>>> 9e3fc93 (yes)
     z_height
     joint_limits_parameters_file
@@ -210,4 +215,5 @@
       </xacro:cylinder_inertial>
     </link>
+<<<<<<< HEAD
     <!-- <xacro:if value="${gripper}">
       <link name="gripper_root_link">
@@ -233,4 +239,6 @@
       </link>
     </xacro:if> -->
+=======
+>>>>>>> 9e3fc93 (yes)
     <!-- joints: main serial chain -->
     <joint name="${prefix}base_link-base_link_inertia" type="fixed">
@@ -242,5 +250,9 @@
            link/frame) to introduce the necessary rotation over Z (of pi rad).
       -->
+<<<<<<< HEAD
       <origin xyz="0 0 ${z_height}" rpy="0 0 ${pi}" />
+=======
+      <origin xyz="0 0 ${z_height}" rpy="0 0 ${pi}" />
+>>>>>>> 9e3fc93 (yes)
     </joint>
     <joint name="${prefix}shoulder_pan_joint" type="revolute">
@@ -316,4 +328,5 @@
       <dynamics damping="0" friction="0"/>
     </joint>
+<<<<<<< HEAD
     <xacro:if value="${gripper}">
       <!-- <joint name="gripper_joint" type="fixed">
@@ -327,4 +340,6 @@
       </xacro:robotiq_hande_gripper>
     </xacro:if>
+=======
+>>>>>>> 9e3fc93 (yes)
     <!-- ROS-Industrial 'base' frame: base_link to UR 'Base' Coordinates transform -->
     <link name="${prefix}base"/>

File: src/fmauch_universal_robot/ur_description/urdf/ur3e.xacro (robot description, xacro)
@@ -15,7 +15,13 @@
   -->
   <!-- <xacro:arg name="z_height" default="$(arg z_h)" /> -->
+<<<<<<< HEAD
   <!-- <xacro:arg name="z_height" default="$(arg z_h)" /> -->
   <xacro:include filename="$(find ur_description)/urdf/inc/ur3e_macro.xacro" >
     <!-- <xacro:arg name="z_height" value="$(arg z_height)" /> -->
+=======
+  <xacro:arg name="z_height" default="$(arg z_h)" />
+  <xacro:include filename="$(find ur_description)/urdf/inc/ur3e_macro.xacro" >
+    <xacro:arg name="z_height" value="$(arg z_height)" />
+>>>>>>> 9e3fc93 (yes)
   </xacro:include>
   <xacro:ur3e_robot prefix="" />

File: src/fmauch_universal_robot/ur_gazebo/urdf/ur.xacro (robot description, xacro)
@@ -43,10 +43,16 @@
   <xacro:arg name="safety_k_position" default="20"/>
   <xacro:arg name="z_height" default="0.0" />
+<<<<<<< HEAD
   <xacro:arg name="gripper" default="false" />
+=======
+>>>>>>> 9e3fc93 (yes)
   <!-- Instantiate the Gazebo robot and pass it all the required arguments. -->
   <xacro:ur_robot_gazebo
     prefix=""
     z_height="$(arg z_height)"
+<<<<<<< HEAD
     gripper="$(arg gripper)"
+=======
+>>>>>>> 9e3fc93 (yes)
     joint_limits_parameters_file="$(arg joint_limit_params)"
     kinematics_parameters_file="$(arg kinematics_params)"

File: src/fmauch_universal_robot/ur_gazebo/urdf/ur_macro.xacro (robot description, xacro)
@@ -34,5 +34,8 @@
    prefix
    z_height
+<<<<<<< HEAD
    gripper
+=======
+>>>>>>> 9e3fc93 (yes)
    joint_limits_parameters_file
    kinematics_parameters_file
@@ -53,5 +56,8 @@
       prefix="${prefix}"
       z_height="${z_height}"
+<<<<<<< HEAD
       gripper="${gripper}"
+=======
+>>>>>>> 9e3fc93 (yes)
       joint_limits_parameters_file="${joint_limits_parameters_file}"
       kinematics_parameters_file="${kinematics_parameters_file}"
