Commit message: Added Gripper

File: src/fmauch_universal_robot/ur_description/urdf/inc/ur_macro.xacro (robot description, xacro)
@@ -44,7 +44,10 @@
   <xacro:include filename="$(find ur_description)/urdf/inc/ur_transmissions.xacro" />
   <xacro:include filename="$(find ur_description)/urdf/inc/ur_common.xacro" />
+  <!-- robotiq_hande_gripper -->
+  <xacro:include filename="$(find robotiq_description)/urdf/robotiq_hande_gripper.urdf.xacro" />
   <xacro:macro name="ur_robot" params="
     prefix
     z_height
+    gripper
     joint_limits_parameters_file
     kinematics_parameters_file
@@ -207,4 +210,27 @@
       </xacro:cylinder_inertial>
     </link>
+    <xacro:if value="${gripper}">
+      <link name="gripper_root_link">
+        <visual>
+          <origin xyz="0 0 0.005" rpy="0 0 0"/>
+          <geometry>
+            <box size="0.01 0.01 0.01"/>
+          </geometry>
+        </visual>
+        <collision>
+          <origin xyz="0 0 0.005" rpy="0 0 0"/>
+          <geometry>
+            <box size="0.01 0.01 0.01"/>
+          </geometry>
+        </collision>
+        <inertial>
+          <mass value="0.01" />
+          <origin xyz="0.0 0.0 0.0" />
+          <inertia ixx = "0.000001" ixy = "0.000000" ixz = "0.000000"
+              iyx = "0.000000" iyy = "0.000001" iyz = "0.000000"
+              izx = "0.000000" izy = "0.000000" izz = "0.000001" />
+        </inertial>
+      </link>
+    </xacro:if>
     <!-- joints: main serial chain -->
     <joint name="${prefix}base_link-base_link_inertia" type="fixed">
@@ -290,4 +316,15 @@
       <dynamics damping="0" friction="0"/>
     </joint>
+    <xacro:if value="${gripper}">
+      <joint name="gripper_joint" type="fixed">
+        <parent link="${prefix}wrist_3_link" />
+        <child link = "gripper_root_link" />
+        <origin xyz="0.0 0.0 0.0" rpy="0.0 0.0 0.0" />
+      </joint>
+      <!-- gripper -->
+      <xacro:robotiq_hande_gripper prefix="" parent="gripper_root_link" >
+        <origin xyz="0.0 0 0.005" rpy="0 0 0"/>
+      </xacro:robotiq_hande_gripper>
+    </xacro:if>
     <!-- ROS-Industrial 'base' frame: base_link to UR 'Base' Coordinates transform -->
     <link name="${prefix}base"/>

File: src/fmauch_universal_robot/ur_gazebo/urdf/ur.xacro (robot description, xacro)
@@ -43,8 +43,10 @@
   <xacro:arg name="safety_k_position" default="20"/>
   <xacro:arg name="z_height" default="0.0" />
+  <xacro:arg name="gripper" default="false" />
   <!-- Instantiate the Gazebo robot and pass it all the required arguments. -->
   <xacro:ur_robot_gazebo
     prefix=""
     z_height="$(arg z_height)"
+    gripper="$(arg gripper)"
     joint_limits_parameters_file="$(arg joint_limit_params)"
     kinematics_parameters_file="$(arg kinematics_params)"

File: src/fmauch_universal_robot/ur_gazebo/urdf/ur_macro.xacro (robot description, xacro)
@@ -34,4 +34,5 @@
    prefix
    z_height
+   gripper
    joint_limits_parameters_file
    kinematics_parameters_file
@@ -52,4 +53,5 @@
       prefix="${prefix}"
       z_height="${z_height}"
+      gripper="${gripper}"
       joint_limits_parameters_file="${joint_limits_parameters_file}"
       kinematics_parameters_file="${kinematics_parameters_file}"

Commit message: gripper attached

File: src/fmauch_universal_robot/ur_description/urdf/inc/ur_macro.xacro (robot description, xacro)
@@ -48,6 +48,6 @@
   <xacro:macro name="ur_robot" params="
     prefix
+    gripper
     z_height
-    gripper
     joint_limits_parameters_file
     kinematics_parameters_file
@@ -210,5 +210,5 @@
       </xacro:cylinder_inertial>
     </link>
-    <xacro:if value="${gripper}">
+    <!-- <xacro:if value="${gripper}">
       <link name="gripper_root_link">
         <visual>
@@ -232,5 +232,5 @@
         </inertial>
       </link>
-    </xacro:if>
+    </xacro:if> -->
     <!-- joints: main serial chain -->
     <joint name="${prefix}base_link-base_link_inertia" type="fixed">
@@ -317,11 +317,11 @@
     </joint>
     <xacro:if value="${gripper}">
-      <joint name="gripper_joint" type="fixed">
+      <!-- <joint name="gripper_joint" type="fixed">
         <parent link="${prefix}wrist_3_link" />
         <child link = "gripper_root_link" />
         <origin xyz="0.0 0.0 0.0" rpy="0.0 0.0 0.0" />
-      </joint>
+      </joint> -->
       <!-- gripper -->
-      <xacro:robotiq_hande_gripper prefix="" parent="gripper_root_link" >
+      <xacro:robotiq_hande_gripper prefix="" parent="${prefix}wrist_3_link" >
         <origin xyz="0.0 0 0.005" rpy="0 0 0"/>
       </xacro:robotiq_hande_gripper>
